File: letItSlide.kicad_pcb (KiCad board)
At the start: 2 copper layers, 285.8 x 84.5 mm, 146 parts, among them SW1 SW_Push, U1 SRV05-4, U2 ATmega32U4-AU, Y1 Crystal_GND24_Small

Commit message: updating repo
cleaning it up a bit
Parts:
- added REF**: Potentiometer_Bourns_PTA4543_Single_Slide, Potentiometer_THT:Potentiometer_Bourns_PTA4543_Single_Slide, F.Cu at (369.1, 75.0)
- added REF**: Potentiometer_Bourns_PTA3043_Single_Slide, Potentiometer_THT:Potentiometer_Bourns_PTA3043_Single_Slide, F.Cu at (341.7, 66.7)
Other:
- net class Default removed
